File: mainboard.kicad_pcb (KiCad board)
At the start: 6 copper layers, 56 x 56 mm, 190 parts, among them J1 USB_C, J2 MCU_SWD, J3 TC_SWD, J4 PMOD_A, J5 PMOD_B, J6 MEZZANINE, Q1 PMOS, Q2 2PNP, SW1 BTN_PROGRAM, SW2 BTN_RESET, SW3 BTN_USER, U1 ECP5-BGA256, U10 W25Q32JVSS, U2 ATSAMD11, U3 PI3USB102G, U4 3V3REG, U5 1V15REG, U6 2V5REG, U7 1V8REG, U8 HyperRAM, U9 USB3343-CP, Y1 Osc60MHz

Commit message: schematic wip
Parts:
- added REF**: C_0201_0603Metric_Pad0.64x0.40mm_HandSolder, Capacitor_SMD:C_0201_0603Metric_Pad0.64x0.40mm_HandSolder, F.Cu at (59.7, 81.5)
- added REF**: C_0201_0603Metric, Capacitor_SMD:C_0201_0603Metric, F.Cu at (63.4, 83.0)
- added REF**: C_0201_0603Metric_Pad0.64x0.40mm_HandSolder, Capacitor_SMD:C_0201_0603Metric_Pad0.64x0.40mm_HandSolder, F.Cu at (61.5, 81.5)
- added REF**: C_0201_0603Metric, Capacitor_SMD:C_0201_0603Metric, F.Cu at (64.8, 83.0)
- added REF**: C_0201_0603Metric, Capacitor_SMD:C_0201_0603Metric, F.Cu at (64.1, 82.3)
Routing:
- net +3V3: track 143.6 -> 131.5 mm, vias 53 -> 49
- net /FPGA Banks 2 and 3/~{BTN_USER}: track 13.5 -> 2.17 mm, vias 1 -> 0
- net GND: track 149.9 -> 145.4 mm, vias 131 -> 130
- net (no net): track 0.00 -> 0.76 mm
