File: analog_supplies.kicad_sch (KiCad schematic)
At the start: 32 parts, among them Q1 PMOS, Q4 2NPN, U24 LDO-ADJ

Commit message: update symbol metadata
Parts:
- FB1: footprint (none) -> Inductor_SMD:L_0603_1608Metric
Changed lines of the file:
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@@
       (effects (font (size 1.27 1.27)))
     )
-    (property "Footprint" "" (at 217.17 48.768 90)
+    (property "Footprint" "Inductor_SMD:L_0603_1608Metric" (at 217.17 48.768 90)
       (effects (font (size 1.27 1.27)) hide)
     )
@@
       (effects (font (size 1.27 1.27)))
     )
-    (property "Footprint" "" (at 217.17 127.508 90)
+    (property "Footprint" "Inductor_SMD:L_0603_1608Metric" (at 217.17 127.508 90)
       (effects (font (size 1.27 1.27)) hide)
     )
@@
       (effects (font (size 1.27 1.27)) (justify left))
     )
-    (property "Footprint" "" (at 46.228 82.55 90)
-      (effects (font (size 1.27 1.27)) hide)
-    )
+    (property "Footprint" "Inductor_SMD:L_0603_1608Metric" (at 46.228 82.55 90)
+      (effects (font (size 1.27 1.27)) hide)
+    )

Commit message: layout wip
Parts:
- C5: footprint Capacitor_SMD:C_0402_1005Metric -> Capacitor_SMD:C_0201_0603Metric; Manufacturer Samsung -> Murata; Part Number CL05B102KB5NNNC -> GRM033R71E102KA01D; Substitution any equivalent -> GRM033R71E102KA01*
Changed lines of the file:
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@@
       (effects (font (size 1.27 1.27)) (justify left))
     )
-    (property "Footprint" "Capacitor_SMD:C_0402_1005Metric" (at 92.4052 96.52 0)
+    (property "Footprint" "Capacitor_SMD:C_0201_0603Metric" (at 92.4052 96.52 0)
       (effects (font (size 1.27 1.27)) hide)
     )
@@
       (effects (font (size 1.27 1.27)) hide)
     )
-    (property "Part Number" "CL05B102KB5NNNC" (at 91.44 92.71 0)
+    (property "Part Number" "GRM033R71E102KA01D" (at 91.44 92.71 0)
       (effects (font (size 1.27 1.27)) hide)
     )
-    (property "Substitution" "any equivalent" (at 91.44 92.71 0)
+    (property "Substitution" "GRM033R71E102KA01*" (at 91.44 92.71 0)
       (effects (font (size 1.27 1.27)) hide)
     )
-    (property "Description" "CAP CER 1000PF 50V X7R 0402" (at 91.44 92.71 0)
+    (property "Description" "CAP CER 1000PF 25V X7R 0201" (at 91.44 92.71 0)
       (effects (font (size 1.27 1.27)) hide)
     )
-    (property "Manufacturer" "Samsung" (at 91.44 92.71 0)
+    (property "Manufacturer" "Murata" (at 91.44 92.71 0)
       (effects (font (size 1.27 1.27)) hide)
     )

Commit message: more layout wip
Parts:
- added Q4: 2NPN, Package_TO_SOT_SMD:SOT-363_SC-70-6, symbol Transistor_BJT:BC847BS
Connections:
- net ~{POWER_GOOD}: now also Q4.1 (E1); no longer Q4.4 (E2)
- net at R28.1: now also Q4.2 (B1); no longer Q4.5 (B2)
- net at R36.2: now also Q4.6 (C1); no longer Q4.3 (C2)
- no-connect marks 0 -> 6
Other:
- moved on the sheet: Q4B
Changed lines of the file:
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@@
   (junction (at 209.55 125.73) (diameter 0) (color 0 0 0 0)
   )
+  (no_connect (at 261.62 78.74))
+  (no_connect (at 261.62 157.48))
+  (no_connect (at 254 73.66))
+  (no_connect (at 261.62 147.32))
+  (no_connect (at 261.62 68.58))
+  (no_connect (at 254 152.4))
   (wire (pts (xy 91.44 87.63) (xy 91.44 88.9))
     (stroke (width 0) (type default))
@@
     )
   )
-  (symbol (lib_id "Transistor_BJT:BC847BS") (at 67.31 111.76 0) (unit 2)
-    (in_bom yes) (on_board yes) (dnp no)
-    (property "Reference" "Q4" (at 72.39 113.6681 0)
-      (effects (font (size 1.27 1.27)) (justify left))
-    )
-    (property "Value" "2NPN" (at 72.39 116.205 0)
-      (effects (font (size 1.27 1.27)) (justify left))
-    )
-    (property "Footprint" "Package_TO_SOT_SMD:SOT-363_SC-70-6" (at 72.39 109.22 0)
-      (effects (font (size 1.27 1.27)) hide)
-    )
-    (property "Datasheet" "https://www.21yangjie.com/pdf/xxh/xxhsjg/BC847BS.pdf" (at 67.31 111.76 0)
-      (effects (font (size 1.27 1.27)) hide)
-    )
-    (property "Manufacturer" "Yangzhou Yangjie" (at 67.31 111.76 0)
-      (effects (font (size 1.27 1.27)) hide)
-    )
-    (property "Part Number" "BC847BS" (at 67.31 111.76 0)
-      (effects (font (size 1.27 1.27)) hide)
-    )
-    (property "Description" "SOT-363 NPN+NPN 0.3W 0.1A 50V" (at 67.31 111.76 0)
+  (symbol (lib_id "Transistor_BJT:BC847BS") (at 207.01 73.66 0) (unit 1)
+    (in_bom yes) (on_board yes) (dnp no) (fields_autoplaced)
+    (property "Reference" "Q4" (at 211.8614 72.8253 0)
+      (effects (font (size 1.27 1.27)) (justify left))
+    )
+    (property "Value" "2NPN" (at 211.8614 75.3622 0)
+      (effects (font (size 1.27 1.27)) (justify left))
+    )
+    (property "Footprint" "Package_TO_SOT_SMD:SOT-363_SC-70-6" (at 212.09 71.12 0)
+      (effects (font (size 1.27 1.27)) hide)
+    )
+    (property "Datasheet" "https://www.21yangjie.com/pdf/xxh/xxhsjg/BC847BS.pdf" (at 207.01 73.66 0)
+      (effects (font (size 1.27 1.27)) hide)
+    )
+    (property "Manufacturer" "Yangzhou Yangjie" (at 207.01 73.66 0)
+      (effects (font (size 1.27 1.27)) hide)
+    )
+    (property "Part Number" "BC847BS" (at 207.01 73.66 0)
+      (effects (font (size 1.27 1.27)) hide)
+    )
+    (property "Description" "SOT-363 NPN+NPN 0.3W 0.1A 50V" (at 207.01 73.66 0)
       (effects (font (size 1.27 1.27)) hide)
     )
@@
       (project "mainboard"
         (path "/fb621148-8145-4217-9712-738e1b5a4823/4ec621be-184d-4855-a96d-f6fa2a788a77/6aa278c8-8281-4438-81b7-90e6d7ac4f12"
+          (reference "Q4") (unit 1)
+        )
+        (path "/fb621148-8145-4217-9712-738e1b5a4823/85575ef9-3107-418a-95d7-1ff02b595e8d"
+          (reference "Q7") (unit 1)
+        )
+      )
+    )
+  )
+  (symbol (lib_id "Transistor_BJT:BC847BS") (at 67.31 111.76 0) (unit 2)
+    (in_bom yes) (on_board yes) (dnp no)
+    (property "Reference" "Q4" (at 72.39 113.6681 0)
+      (effects (font (size 1.27 1.27)) (justify left))
+    )
+    (property "Value" "2NPN" (at 72.39 116.205 0)
+      (effects (font (size 1.27 1.27)) (justify left))
+    )
+    (property "Footprint" "Package_TO_SOT_SMD:SOT-363_SC-70-6" (at 72.39 109.22 0)
+      (effects (font (size 1.27 1.27)) hide)
+    )
+    (property "Datasheet" "https://www.21yangjie.com/pdf/xxh/xxhsjg/BC847BS.pdf" (at 67.31 111.76 0)
+      (effects (font (size 1.27 1.27)) hide)
+    )
+    (property "Manufacturer" "Yangzhou Yangjie" (at 67.31 111.76 0)
+      (effects (font (size 1.27 1.27)) hide)
+    )
+    (property "Part Number" "BC847BS" (at 67.31 111.76 0)
+      (effects (font (size 1.27 1.27)) hide)
+    )
+    (property "Description" "SOT-363 NPN+NPN 0.3W 0.1A 50V" (at 67.31 111.76 0)
+      (effects (font (size 1.27 1.27)) hide)
+    )
+    (pin "1")
+    (pin "2")
+    (pin "6")
+    (pin "3")
+    (pin "4")
+    (pin "5")
+    (instances
+      (project "mainboard"
+        (path "/fb621148-8145-4217-9712-738e1b5a4823/4ec621be-184d-4855-a96d-f6fa2a788a77/6aa278c8-8281-4438-81b7-90e6d7ac4f12"
           (reference "Q4") (unit 2)
         )
@@
         (path "/fb621148-8145-4217-9712-738e1b5a4823/85575ef9-3107-418a-95d7-1ff02b595e8d"
           (reference "FB2") (unit 1)
+        )
+      )
+    )
+  )
+  (symbol (lib_id "Transistor_BJT:BC847BS") (at 259.08 73.66 0) (unit 2)
+    (in_bom yes) (on_board yes) (dnp no)
+    (property "Reference" "Q4" (at 264.16 75.5681 0)
+      (effects (font (size 1.27 1.27)) (justify left))
+    )
+    (property "Value" "2NPN" (at 264.16 78.105 0)
+      (effects (font (size 1.27 1.27)) (justify left))
+    )
+    (property "Footprint" "Package_TO_SOT_SMD:SOT-363_SC-70-6" (at 264.16 71.12 0)
+      (effects (font (size 1.27 1.27)) hide)
+    )
+    (property "Datasheet" "https://www.21yangjie.com/pdf/xxh/xxhsjg/BC847BS.pdf" (at 259.08 73.66 0)
+      (effects (font (size 1.27 1.27)) hide)
+    )
+    (property "Manufacturer" "Yangzhou Yangjie" (at 259.08 73.66 0)
+      (effects (font (size 1.27 1.27)) hide)
+    )
+    (property "Part Number" "BC847BS" (at 259.08 73.66 0)
+      (effects (font (size 1.27 1.27)) hide)
+    )
+    (property "Description" "SOT-363 NPN+NPN 0.3W 0.1A 50V" (at 259.08 73.66 0)
+      (effects (font (size 1.27 1.27)) hide)
+    )
+    (pin "1")
+    (pin "2")
+    (pin "6")
+    (pin "3")
+    (pin "4")
+    (pin "5")
+    (instances
+      (project "mainboard"
+        (path "/fb621148-8145-4217-9712-738e1b5a4823/4ec621be-184d-4855-a96d-f6fa2a788a77/6aa278c8-8281-4438-81b7-90e6d7ac4f12"
+          (reference "Q4") (unit 2)
+        )
+        (path "/fb621148-8145-4217-9712-738e1b5a4823/4ec621be-184d-4855-a96d-f6fa2a788a77/90da2209-0e18-4bd4-8ef6-3d6f9ed46ff8"
+          (reference "Q4") (unit 2)
+        )
+        (path "/fb621148-8145-4217-9712-738e1b5a4823/85575ef9-3107-418a-95d7-1ff02b595e8d"
+          (reference "Q7") (unit 2)
         )
       )
@@
     )
   )
-  (symbol (lib_id "Transistor_BJT:BC847BS") (at 207.01 73.66 0) (unit 2)
+  (symbol (lib_id "Transistor_BJT:BC847BS") (at 259.08 152.4 0) (unit 2)
     (in_bom yes) (on_board yes) (dnp no)
-    (property "Reference" "Q4" (at 212.09 75.5681 0)
-      (effects (font (size 1.27 1.27)) (justify left))
-    )
-    (property "Value" "2NPN" (at 212.09 78.105 0)
-      (effects (font (size 1.27 1.27)) (justify left))
-    )
-    (property "Footprint" "Package_TO_SOT_SMD:SOT-363_SC-70-6" (at 212.09 71.12 0)
-      (effects (font (size 1.27 1.27)) hide)
-    )
-    (property "Datasheet" "https://www.21yangjie.com/pdf/xxh/xxhsjg/BC847BS.pdf" (at 207.01 73.66 0)
-      (effects (font (size 1.27 1.27)) hide)
-    )
-    (property "Manufacturer" "Yangzhou Yangjie" (at 207.01 73.66 0)
-      (effects (font (size 1.27 1.27)) hide)
-    )
-    (property "Part Number" "BC847BS" (at 207.01 73.66 0)
-      (effects (font (size 1.27 1.27)) hide)
-    )
-    (property "Description" "SOT-363 NPN+NPN 0.3W 0.1A 50V" (at 207.01 73.66 0)
-      (effects (font (size 1.27 1.27)) hide)
-    )
+    (property "Reference" "Q4" (at 264.16 154.3081 0)
+      (effects (font (size 1.27 1.27)) (justify left))
+    )
+    (property "Value" "2NPN" (at 264.16 156.845 0)
+      (effects (font (size 1.27 1.27)) (justify left))
+    )
+    (property "Footprint" "Package_TO_SOT_SMD:SOT-363_SC-70-6" (at 264.16 149.86 0)
+      (effects (font (size 1.27 1.27)) hide)
+    )
+    (property "Datasheet" "https://www.21yangjie.com/pdf/xxh/xxhsjg/BC847BS.pdf" (at 259.08 152.4 0)
+      (effects (font (size 1.27 1.27)) hide)
+    )
+    (property "Manufacturer" "Yangzhou Yangjie" (at 259.08 152.4 0)
+      (effects (font (size 1.27 1.27)) hide)
+    )
+    (property "Part Number" "BC847BS" (at 259.08 152.4 0)
+      (effects (font (size 1.27 1.27)) hide)
+    )
+    (property "Description" "SOT-363 NPN+NPN 0.3W 0.1A 50V" (at 259.08 152.4 0)
+      (effects (font (size 1.27 1.27)) hide)
+    )
