File: radio.kicad_sch (KiCad schematic)
At the start: 44 parts, among them U11 MAX5865

Commit message: passive component selections
Parts:
- C92: Manufacturer (none) -> Murata; Part Number (none) -> GRM033R60J473KE19D; Substitution (none) -> GRM033R60J473KE19*
- R112, R113, R56, R57: Manufacturer (none) -> Yageo; Part Number (none) -> RC0201JR-07820RL; Substitution (none) -> any equivalent
Changed lines of the file:
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@@
+      (effects (font (size 1.27 1.27)) hide)
+    )
+    (property "Description" "RES 820 OHM 5% 1/20W 0201" (at 168.91 95.25 0)
+      (effects (font (size 1.27 1.27)) hide)
+    )
+    (property "Manufacturer" "Yageo" (at 168.91 95.25 0)
+      (effects (font (size 1.27 1.27)) hide)
+    )
+    (property "Part Number" "RC0201JR-07820RL" (at 168.91 95.25 0)
+      (effects (font (size 1.27 1.27)) hide)
+    )
+    (property "Substitution" "any equivalent" (at 168.91 95.25 0)
       (effects (font (size 1.27 1.27)) hide)
     )
@@
       (effects (font (size 1.27 1.27)) hide)
     )
+    (property "Description" "RES 820 OHM 5% 1/20W 0201" (at 158.75 95.25 0)
+      (effects (font (size 1.27 1.27)) hide)
+    )
+    (property "Manufacturer" "Yageo" (at 158.75 95.25 0)
+      (effects (font (size 1.27 1.27)) hide)
+    )
+    (property "Part Number" "RC0201JR-07820RL" (at 158.75 95.25 0)
+      (effects (font (size 1.27 1.27)) hide)
+    )
+    (property "Substitution" "any equivalent" (at 158.75 95.25 0)
+      (effects (font (size 1.27 1.27)) hide)
+    )
     (pin "1")
     (pin "2")
@@
     )
     (property "Datasheet" "~" (at 191.77 67.31 0)
+      (effects (font (size 1.27 1.27)) hide)
+    )
+    (property "Description" "CAP CER 0.047UF 6.3V X5R 0201" (at 191.77 67.31 0)
+      (effects (font (size 1.27 1.27)) hide)
+    )
+    (property "Manufacturer" "Murata" (at 191.77 67.31 0)
+      (effects (font (size 1.27 1.27)) hide)
+    )
+    (property "Part Number" "GRM033R60J473KE19D" (at 191.77 67.31 0)
+      (effects (font (size 1.27 1.27)) hide)
+    )
+    (property "Substitution" "GRM033R60J473KE19*" (at 191.77 67.31 0)
       (effects (font (size 1.27 1.27)) hide)
     )
@@
       (effects (font (size 1.27 1.27)) hide)
     )
+    (property "Description" "RES 820 OHM 5% 1/20W 0201" (at 148.59 95.25 0)
+      (effects (font (size 1.27 1.27)) hide)
+    )
+    (property "Manufacturer" "Yageo" (at 148.59 95.25 0)
+      (effects (font (size 1.27 1.27)) hide)
+    )
+    (property "Part Number" "RC0201JR-07820RL" (at 148.59 95.25 0)
+      (effects (font (size 1.27 1.27)) hide)
+    )
+    (property "Substitution" "any equivalent" (at 148.59 95.25 0)
+      (effects (font (size 1.27 1.27)) hide)
+    )
     (pin "1")
     (pin "2")
@@
     )
     (property "Datasheet" "~" (at 191.77 82.55 0)
+      (effects (font (size 1.27 1.27)) hide)
+    )
+    (property "Description" "CAP CER 0.047UF 6.3V X5R 0201" (at 191.77 82.55 0)
+      (effects (font (size 1.27 1.27)) hide)
+    )
+    (property "Manufacturer" "Murata" (at 191.77 82.55 0)
+      (effects (font (size 1.27 1.27)) hide)
+    )
+    (property "Part Number" "GRM033R60J473KE19D" (at 191.77 82.55 0)
+      (effects (font (size 1.27 1.27)) hide)
+    )
+    (property "Substitution" "GRM033R60J473KE19*" (at 191.77 82.55 0)
       (effects (font (size 1.27 1.27)) hide)
     )
@@
       (effects (font (size 1.27 1.27)) hide)
     )
+    (property "Description" "RES 820 OHM 5% 1/20W 0201" (at 138.43 95.25 0)
+      (effects (font (size 1.27 1.27)) hide)
+    )
+    (property "Manufacturer" "Yageo" (at 138.43 95.25 0)
+      (effects (font (size 1.27 1.27)) hide)
+    )
+    (property "Part Number" "RC0201JR-07820RL" (at 138.43 95.25 0)
+      (effects (font (size 1.27 1.27)) hide)
+    )
+    (property "Substitution" "any equivalent" (at 138.43 95.25 0)
+      (effects (font (size 1.27 1.27)) hide)
+    )
     (pin "1")
     (pin "2")
@@
     )
     (property "Datasheet" "~" (at 191.77 74.93 0)
+      (effects (font (size 1.27 1.27)) hide)
+    )
+    (property "Description" "CAP CER 0.047UF 6.3V X5R 0201" (at 191.77 74.93 0)
+      (effects (font (size 1.27 1.27)) hide)
+    )
+    (property "Manufacturer" "Murata" (at 191.77 74.93 0)
+      (effects (font (size 1.27 1.27)) hide)
+    )
+    (property "Part Number" "GRM033R60J473KE19D" (at 191.77 74.93 0)
+      (effects (font (size 1.27 1.27)) hide)
+    )
+    (property "Substitution" "GRM033R60J473KE19*" (at 191.77 74.93 0)
       (effects (font (size 1.27 1.27)) hide)
     )
@@
       (effects (font (size 1.27 1.27)) hide)
     )
+    (property "Description" "CAP CER 0.047UF 6.3V X5R 0201" (at 191.77 90.17 0)
+      (effects (font (size 1.27 1.27)) hide)
+    )
+    (property "Manufacturer" "Murata" (at 191.77 90.17 0)
+      (effects (font (size 1.27 1.27)) hide)
+    )
+    (property "Part Number" "GRM033R60J473KE19D" (at 191.77 90.17 0)
+      (effects (font (size 1.27 1.27)) hide)
+    )
+    (property "Substitution" "GRM033R60J473KE19*" (at 191.77 90.17 0)
+      (effects (font (size 1.27 1.27)) hide)
+    )
